File: hardware/kicad/Automatrix_PVDG_RevA.kicad_sch (KiCad schematic)
At the start: 0 parts

Commit message: hw: persist KiCad 10 validated Rev-A sources
Parts:
- added BT1: CR1220, Battery:BatteryHolder_Keystone_3000_1x12mm, symbol Automatrix:BAT
- added C3_BOOT, C3_IN2, C_BOOT1: 0.1uF 50V, Capacitor_SMD:C_0603_1608Metric, symbol Automatrix:C
- added C3_FB: 100pF, Capacitor_SMD:C_0603_1608Metric, symbol Automatrix:C
- added C3_IN1: 10uF 35V, Capacitor_SMD:C_1206_3216Metric, symbol Automatrix:C_BIG
- added C3_OUT1, C3_OUT2: 22uF 25V, Capacitor_SMD:C_1206_3216Metric, symbol Automatrix:C_BIG
- added CIN1, CIN2: 2.2uF 100V, Capacitor_SMD:C_1210_3225Metric, symbol Automatrix:C_BIG
- added CINB: 100uF 50V, Capacitor_THT:CP_Radial_D10.0mm_P5.00mm, symbol Automatrix:C_BIG
- added COUT1, COUT2: 47uF 10V, Capacitor_SMD:C_1210_3225Metric, symbol Automatrix:C_BIG
- added COUT3, C_MCU2, C_SD2: 0.1uF, Capacitor_SMD:C_0603_1608Metric, symbol Automatrix:C
- added C_1V2: 10nF, Capacitor_SMD:C_0603_1608Metric, symbol Automatrix:C
- added C_COMP: 6.8nF, Capacitor_SMD:C_0603_1608Metric, symbol Automatrix:C
- added C_COMP_HF: 39pF, Capacitor_SMD:C_0603_1608Metric, symbol Automatrix:C
- added C_EN: 1uF, Capacitor_SMD:C_0603_1608Metric, symbol Automatrix:C
- added C_MCU1, C_SD1: 10uF, Capacitor_SMD:C_0805_2012Metric, symbol Automatrix:C_BIG
- added C_RS2321, C_RS2322, C_RS2323, C_RS2324, C_RS2325: 0.1uF DNP, Capacitor_SMD:C_0603_1608Metric, symbol Automatrix:CAP
- added C_TOCAP: 4.7uF, Capacitor_SMD:C_0805_2012Metric, symbol Automatrix:C_BIG
- added C_XI, C_XO: 18pF, Capacitor_SMD:C_0603_1608Metric, symbol Automatrix:C
- added DTVS1: SMBJ33A, Diode_SMD:D_SMA, symbol Automatrix:TVS
- added DZREV: 12V gate clamp, Diode_SMD:D_SOD-123, symbol Automatrix:ZENER
- added D_DI1, D_DI2, D_DI3, D_DI4: 1N4148 reverse, Diode_SMD:D_SOD-123, symbol Automatrix:DIODE
- added D_FLY1, D_FLY2, D_FLY3, D_FLY4: SS14, Diode_SMD:D_SMA, symbol Automatrix:DIODE
- added D_LED1: RELAY1, LED_SMD:LED_0805_2012Metric, symbol Automatrix:LED
- added D_LED2: RELAY2, LED_SMD:LED_0805_2012Metric, symbol Automatrix:LED
- added D_LED3: RELAY3, LED_SMD:LED_0805_2012Metric, symbol Automatrix:LED
- added D_LED4: RELAY4, LED_SMD:LED_0805_2012Metric, symbol Automatrix:LED
- added D_OR_FIELD, D_OR_USB: SS34, Diode_SMD:D_SMA, symbol Automatrix:DIODE
- added D_RS485A_TVS, D_RS485B_TVS: SM712, Package_TO_SOT_SMD:SOT-23, symbol Automatrix:TVS
- added D_RTC_BAT, D_RTC_MAIN: BAT54, Diode_SMD:D_SOD-323, symbol Automatrix:DIODE
- added D_STATUS: STATUS, LED_SMD:LED_0805_2012Metric, symbol Automatrix:LED
- added D_USB_DN, D_USB_DP: USB ESD, Package_TO_SOT_SMD:SOT-23, symbol Automatrix:TVS
- added F1: 3.15A 60V+, Fuse:Fuse_1206_3216Metric, symbol Automatrix:FUSE
- added F_HMI: 1.1A PTC, Fuse:Fuse_1206_3216Metric, symbol Automatrix:FUSE
- added J_DI: DI1-4/COM, TerminalBlock_CUI:TerminalBlock_CUI_TB007-508-05_1x05_P5.08mm_Horizontal, symbol Automatrix:CONN5
- added J_ETH: J1B1211CCD, Connector_RJ:RJ45_Cetus_J1B1211CCD_Horizontal, symbol Automatrix:MAGJACK
- added J_HMI: HMI +5/GND/TX/RX, Connector_JST:JST_XH_B4B-XH-A_1x04_P2.50mm_Vertical, symbol Automatrix:CONN4
- added J_PWR: 12/24V FIELD IN, TerminalBlock_CUI:TerminalBlock_CUI_TB007-508-02_1x02_P5.08mm_Horizontal, symbol Automatrix:CONN2
- added J_RLY1: Relay1 NC/COM/NO, TerminalBlock_CUI:TerminalBlock_CUI_TB007-508-03_1x03_P5.08mm_Horizontal, symbol Automatrix:CONN3
- added J_RLY2: Relay2 NC/COM/NO, TerminalBlock_CUI:TerminalBlock_CUI_TB007-508-03_1x03_P5.08mm_Horizontal, symbol Automatrix:CONN3
- added J_RLY3: Relay3 NC/COM/NO, TerminalBlock_CUI:TerminalBlock_CUI_TB007-508-03_1x03_P5.08mm_Horizontal, symbol Automatrix:CONN3
- added J_RLY4: Relay4 NC/COM/NO, TerminalBlock_CUI:TerminalBlock_CUI_TB007-508-03_1x03_P5.08mm_Horizontal, symbol Automatrix:CONN3
- added J_RS232: RS232 GND/TX/RX DNP, Connector_JST:JST_XH_B3B-XH-A_1x03_P2.50mm_Vertical, symbol Automatrix:CONN3
- added J_RS485A: RS485A A/B/GND, TerminalBlock_CUI:TerminalBlock_CUI_TB007-508-03_1x03_P5.08mm_Horizontal, symbol Automatrix:CONN3
- added J_RS485B: RS485B A/B/GND, TerminalBlock_CUI:TerminalBlock_CUI_TB007-508-03_1x03_P5.08mm_Horizontal, symbol Automatrix:CONN3
- added J_SD: microSD DNP, Connector_Card:microSD_HC_Hirose_DM3AT-SF-PEJM5, symbol Automatrix:SD
- added J_USB: USB-C SERVICE, Connector_USB:USB_C_Receptacle_GCT_USB4105-xx-A_16P_TopMnt_Horizontal, symbol Automatrix:USB_C
- added K1, K2, K3, K4: HF3FF/005-1ZST, Relay_THT:Relay_SPDT_Hongfa_JQC-3FF_0XX-1Z, symbol Automatrix:RELAY
- added L1: 8.2uH >=5A, Inductor_SMD:L_Wuerth_XHMI-6060, symbol Automatrix:L
- added L2: 6.8uH 5A, Inductor_SMD:L_Wuerth_XHMI-6060, symbol Automatrix:L
- added Q1, Q2, Q3, Q4: AO3400A, Package_TO_SOT_SMD:SOT-23, symbol Automatrix:NMOS
- added QREV: DMP6023LSS, Package_SO:SO-8_3.9x4.9mm_P1.27mm, symbol Automatrix:PMOS
- added RREV, R_PD1, R_PD2, R_PD3, R_PD4: 100k, Resistor_SMD:R_0603_1608Metric, symbol Automatrix:R
- added R_BOOT, R_DIPU1, R_DIPU2, R_DIPU3, R_DIPU4, R_EN, R_HMIRX_TOP, R_PM0, R_PM1, R_PM2, R_RS485A_DE, R_RS485B_DE, R_SDCS, R_SDMISO, R_SDMOSI, R_SDSCLK: 10k, Resistor_SMD:R_0603_1608Metric, symbol Automatrix:R
- added R_CC1, R_CC2: 5.1k, Resistor_SMD:R_0603_1608Metric, symbol Automatrix:R
- added R_COMP: 13k, Resistor_SMD:R_0603_1608Metric, symbol Automatrix:R
- added R_DI1, R_DI2, R_DI3, R_DI4: 3.3k 0.25W, Resistor_SMD:R_1206_3216Metric, symbol Automatrix:R
- added R_EN1: 523k, Resistor_SMD:R_0603_1608Metric, symbol Automatrix:R
- added R_EN2: 84.5k, Resistor_SMD:R_0603_1608Metric, symbol Automatrix:R
- added R_EXRES: 12.4k 1%, Resistor_SMD:R_0603_1608Metric, symbol Automatrix:R
- added R_FB1: 53.6k, Resistor_SMD:R_0603_1608Metric, symbol Automatrix:R
- added R_FB2: 10.2k, Resistor_SMD:R_0603_1608Metric, symbol Automatrix:R
- added R_G1, R_G2, R_G3, R_G4, R_HMITX: 100R, Resistor_SMD:R_0603_1608Metric, symbol Automatrix:R
- added R_HMIRX_BOT: 20k, Resistor_SMD:R_0603_1608Metric, symbol Automatrix:R
- added R_LED1, R_LED2, R_LED3, R_LED4, R_STATUS: 1k, Resistor_SMD:R_0603_1608Metric, symbol Automatrix:R
- added R_RS485A_BIASA, R_RS485A_BIASB, R_RS485B_BIASA, R_RS485B_BIASB: 680R DNP, Resistor_SMD:R_0603_1608Metric, symbol Automatrix:R
- added R_RS485A_TERM, R_RS485B_TERM: 120R DNP, Resistor_SMD:R_1206_3216Metric, symbol Automatrix:R
- added R_RT: 162k, Resistor_SMD:R_0603_1608Metric, symbol Automatrix:R
- added R_SCL, R_SDA: 4.7k, Resistor_SMD:R_0603_1608Metric, symbol Automatrix:R
- added R_XTAL: 1M, Resistor_SMD:R_0603_1608Metric, symbol Automatrix:R
- added SW_BOOT: BOOT, Button_Switch_SMD:Panasonic_EVQPUJ_EVQPUA, symbol Automatrix:SW
- added SW_RESET: RESET, Button_Switch_SMD:Panasonic_EVQPUJ_EVQPUA, symbol Automatrix:SW
- added U1: ESP32-S3-WROOM-1-N8, RF_Module:ESP32-S3-WROOM-1, symbol Automatrix:ESP32S3
- added U2: W5500, Package_QFP:LQFP-48_7x7mm_P0.5mm, symbol Automatrix:W5500
- added U3, U4: THVD1410D, Package_SO:SOIC-8_3.9x4.9mm_P1.27mm, symbol Automatrix:THVD1410
- added U5: TPS54360B, Package_SO:TI_SO-PowerPAD-8_ThermalVias, symbol Automatrix:TPS54360B
- added U6: AP63203WU-7, Package_TO_SOT_SMD:TSOT-23-6, symbol Automatrix:AP63203
- added U7: MAX3232 DNP, Package_SO:SOIC-16_3.9x9.9mm_P1.27mm, symbol Automatrix:MAX3232
- added U_DI1, U_DI2, U_DI3, U_DI4: LTV-817, Package_DIP:DIP-4_W7.62mm, symbol Automatrix:OPTO
- added U_RTC: PCF8563T DNP, Package_SO:SOIC-8_3.9x4.9mm_P1.27mm, symbol Automatrix:PCF8563
- added Y1: 25MHz, Crystal:Crystal_SMD_3225-4Pin_3.2x2.5mm, symbol Automatrix:CRYSTAL2
- added Y_RTC: 32.768kHz, Crystal:Crystal_SMD_3215-2Pin_3.2x1.5mm, symbol Automatrix:CRYSTAL2
Connections:
- new net 3V3: C3_FB.1, C3_OUT1.1 (+), C3_OUT2.1 (+), C_MCU1.1 (+), C_MCU2.1, C_RS2325.1, C_SD1.1 (+), C_SD2.1, D_RTC_MAIN.2 (A), J_ETH.10 (CT_TX), J_ETH.11 (CT_RX), J_ETH.6 (LED_LINK_A)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
- new net 5V_FIELD: COUT1.1 (+), COUT2.1 (+), COUT3.1, D_FLY1.1 (K), D_FLY2.1 (K), D_FLY3.1 (K), D_FLY4.1 (K), D_OR_FIELD.2 (A), F_HMI.1, K1.A1 (COIL_A), K2.A1 (COIL_A), K3.A1 (COIL_A)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
- new net 5V_HMI: F_HMI.2, J_HMI.1 (Pin_1)
- new net 5V_LOGIC_IN: C3_IN1.1 (+), C3_IN2.1, D_OR_FIELD.1 (K), D_OR_USB.1 (K), U6.2 (EN), U6.3 (VIN)
- new net BUCK3_BST: C3_BOOT.1, U6.6 (BST)
- new net BUCK3_SW: C3_BOOT.2, L2.1, U6.5 (SW)
- new net BUCK_BOOT: C_BOOT1.1, U5.1 (BOOT)
- new net BUCK_COMP: C_COMP_HF.1, R_COMP.1, U5.6 (COMP)
- new net BUCK_COMP_RC: C_COMP.1, R_COMP.2
- new net BUCK_EN: R_EN1.2, R_EN2.1, U5.3 (EN)
- new net BUCK_FB: R_FB1.2, R_FB2.1, U5.5 (FB)
- new net BUCK_RT: R_RT.1, U5.4 (RT_CLK)
- new net BUCK_SW: C_BOOT1.2, L1.1, U5.8 (SW)
- new net CHASSIS: J_ETH.12 (CHASSIS), J_ETH.9 (SHIELD), J_USB.SH (SHIELD)
- new net DI1_FIELD: J_DI.1 (Pin_1), R_DI1.1
- new net DI1_LEDK: D_DI1.1 (K), R_DI1.2, U_DI1.1 (A)
- new net DI1_LOGIC: R_DIPU1.2, U1.39 (IO1), U_DI1.4 (C)
- new net DI2_FIELD: J_DI.2 (Pin_2), R_DI2.1
- new net DI2_LEDK: D_DI2.1 (K), R_DI2.2, U_DI2.1 (A)
- new net DI2_LOGIC: R_DIPU2.2, U1.38 (IO2), U_DI2.4 (C)
- new net DI3_FIELD: J_DI.3 (Pin_3), R_DI3.1
- new net DI3_LEDK: D_DI3.1 (K), R_DI3.2, U_DI3.1 (A)
- new net DI3_LOGIC: R_DIPU3.2, U1.24 (IO47), U_DI3.4 (C)
- new net DI4_FIELD: J_DI.4 (Pin_4), R_DI4.1
- new net DI4_LEDK: D_DI4.1 (K), R_DI4.2, U_DI4.1 (A)
- new net DI4_LOGIC: R_DIPU4.2, U1.25 (IO48), U_DI4.4 (C)
- new net DI_COM: D_DI1.2 (A), D_DI2.2 (A), D_DI3.2 (A), D_DI4.2 (A), J_DI.5 (Pin_5), U_DI1.2 (K), U_DI2.2 (K), U_DI3.2 (K), U_DI4.2 (K)
- new net ESP_BOOT: R_BOOT.2, SW_BOOT.1, U1.27 (IO0)
- new net ESP_EN: C_EN.1, R_EN.2, SW_RESET.1, U1.3 (EN)
- new net ETH_1V2: C_1V2.1, U2.22 (1V2O)
- new net ETH_CS: U1.18 (IO10), U2.32 (SCSn)
- new net ETH_EXRES: R_EXRES.1, U2.10 (EXRES1)
- new net ETH_INT: U1.17 (IO9), U2.36 (INTn)
- new net ETH_LED_ACT: J_ETH.7 (LED_ACT_K), U2.27 (ACTLED)
- new net ETH_LED_LINK: J_ETH.5 (LED_LINK_K), U2.25 (LINKLED)
- new net ETH_MISO: U1.21 (IO13), U2.34 (MISO)
- new net ETH_MOSI: U1.19 (IO11), U2.35 (MOSI)
- new net ETH_PMODE0: R_PM0.2, U2.45 (PMODE0)
- new net ETH_PMODE1: R_PM1.2, U2.44 (PMODE1)
- new net ETH_PMODE2: R_PM2.2, U2.43 (PMODE2)
- new net ETH_RST: U1.12 (IO8), U2.37 (RSTn)
- new net ETH_RXN: J_ETH.4 (PHY_RXN), U2.5 (RXN)
- new net ETH_RXP: J_ETH.3 (PHY_RXP), U2.6 (RXP)
- new net ETH_SCLK: U1.20 (IO12), U2.33 (SCLK)
- new net ETH_TOCAP: C_TOCAP.1 (+), U2.20 (TOCAP)
- new net ETH_TXN: J_ETH.2 (PHY_TXN), U2.1 (TXN)
- new net ETH_TXP: J_ETH.1 (PHY_TXP), U2.2 (TXP)
- new net ETH_XI: C_XI.1, R_XTAL.1, U2.30 (XI_CLKIN), Y1.1
- new net ETH_XO: C_XO.1, R_XTAL.2, U2.31 (XO), Y1.2
- new net GND: BT1.2 (-), C3_FB.2, C3_IN1.2 (-), C3_IN2.2, C3_OUT1.2 (-), C3_OUT2.2 (-), CIN1.2 (-), CIN2.2 (-), CINB.2 (-), COUT1.2 (-), COUT2.2 (-), COUT3.2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
- new net HMI_RS232_RX: J_RS232.3 (Pin_3), U7.13 (R1IN)
- new net HMI_RS232_TX: J_RS232.2 (Pin_2), U7.14 (T1OUT)
- new net HMI_RX: R_HMIRX_BOT.1, R_HMIRX_TOP.2, U1.22 (IO14), U7.12 (R1OUT)
- new net HMI_RX_IN: J_HMI.4 (Pin_4), R_HMIRX_TOP.1
- new net HMI_TX: R_HMITX.1, U1.8 (IO15), U7.11 (T1IN)
- new net HMI_TX_OUT: J_HMI.3 (Pin_3), R_HMITX.2
- new net RELAY1_COIL: D_FLY1.2 (A), D_LED1.1 (K), K1.A2 (COIL_B), Q1.3 (D)
- new net RELAY1_CTL: R_G1.1, U1.4 (IO4)
- new net RELAY1_GATE: Q1.1 (G), R_G1.2, R_PD1.1
- new net RELAY2_COIL: D_FLY2.2 (A), D_LED2.1 (K), K2.A2 (COIL_B), Q2.3 (D)
- new net RELAY2_CTL: R_G2.1, U1.5 (IO5)
- new net RELAY2_GATE: Q2.1 (G), R_G2.2, R_PD2.1
- new net RELAY3_COIL: D_FLY3.2 (A), D_LED3.1 (K), K3.A2 (COIL_B), Q3.3 (D)
- new net RELAY3_CTL: R_G3.1, U1.6 (IO6)
- new net RELAY3_GATE: Q3.1 (G), R_G3.2, R_PD3.1
- new net RELAY4_COIL: D_FLY4.2 (A), D_LED4.1 (K), K4.A2 (COIL_B), Q4.3 (D)
- new net RELAY4_CTL: R_G4.1, U1.7 (IO7)
- new net RELAY4_GATE: Q4.1 (G), R_G4.2, R_PD4.1
- new net REV_GATE: DZREV.2 (A), QREV.1 (G), RREV.1
- new net RLY1_COM: J_RLY1.2 (Pin_2), K1.11 (COM)
- new net RLY1_LED_A: D_LED1.2 (A), R_LED1.2
- new net RLY1_NC: J_RLY1.1 (Pin_1), K1.12 (NC)
- new net RLY1_NO: J_RLY1.3 (Pin_3), K1.14 (NO)
- new net RLY2_COM: J_RLY2.2 (Pin_2), K2.11 (COM)
- new net RLY2_LED_A: D_LED2.2 (A), R_LED2.2
- new net RLY2_NC: J_RLY2.1 (Pin_1), K2.12 (NC)
- new net RLY2_NO: J_RLY2.3 (Pin_3), K2.14 (NO)
- new net RLY3_COM: J_RLY3.2 (Pin_2), K3.11 (COM)
- new net RLY3_LED_A: D_LED3.2 (A), R_LED3.2
- new net RLY3_NC: J_RLY3.1 (Pin_1), K3.12 (NC)
- new net RLY3_NO: J_RLY3.3 (Pin_3), K3.14 (NO)
- new net RLY4_COM: J_RLY4.2 (Pin_2), K4.11 (COM)
- new net RLY4_LED_A: D_LED4.2 (A), R_LED4.2
- new net RLY4_NC: J_RLY4.1 (Pin_1), K4.12 (NC)
- new net RLY4_NO: J_RLY4.3 (Pin_3), K4.14 (NO)
- new net RS232_C1M: C_RS2321.2, U7.3 (C1-)
- new net RS232_C1P: C_RS2321.1, U7.1 (C1+)
- new net RS232_C2M: C_RS2322.2, U7.5 (C2-)
- new net RS232_C2P: C_RS2322.1, U7.4 (C2+)
- new net RS232_VMINUS: C_RS2324.1, U7.6 (V-)
- new net RS232_VPLUS: C_RS2323.1, U7.2 (V+)
- new net RS485A_A: D_RS485A_TVS.1 (A), J_RS485A.1 (Pin_1), R_RS485A_BIASA.2, R_RS485A_TERM.1, U3.6 (A)
- new net RS485A_B: D_RS485A_TVS.2 (K), J_RS485A.2 (Pin_2), R_RS485A_BIASB.1, R_RS485A_TERM.2, U3.7 (B)
- new net RS485A_DE: R_RS485A_DE.1, U1.35 (IO42), U3.2 (REn), U3.3 (DE)
- new net RS485A_RX: U1.36 (IO44), U3.1 (R)
- new net RS485A_TX: U1.37 (IO43), U3.4 (D)
- new net RS485B_A: D_RS485B_TVS.1 (A), J_RS485B.1 (Pin_1), R_RS485B_BIASA.2, R_RS485B_TERM.1, U4.6 (A)
- new net RS485B_B: D_RS485B_TVS.2 (K), J_RS485B.2 (Pin_2), R_RS485B_BIASB.1, R_RS485B_TERM.2, U4.7 (B)
- new net RS485B_DE: R_RS485B_DE.1, U1.9 (IO16), U4.2 (REn), U4.3 (DE)
- new net RS485B_RX: U1.11 (IO18), U4.1 (R)
- new net RS485B_TX: U1.10 (IO17), U4.4 (D)
- new net RTC_BAT: BT1.1 (+), D_RTC_BAT.2 (A)
- new net RTC_SCL: R_SCL.2, U1.32 (IO39), U_RTC.6 (SCL)
- new net RTC_SDA: R_SDA.2, U1.31 (IO38), U_RTC.5 (SDA)
- new net RTC_VDD: D_RTC_BAT.1 (K), D_RTC_MAIN.1 (K), U_RTC.8 (VDD)
- new net RTC_X1: U_RTC.1 (OSCI), Y_RTC.1
- new net RTC_X2: U_RTC.2 (OSCO), Y_RTC.2
- new net SD_CS: J_SD.2 (CS_DAT3), R_SDCS.2, U1.29 (IO36)
- new net SD_MISO: J_SD.7 (MISO_DAT0), R_SDMISO.2, U1.30 (IO37)
- new net SD_MOSI: J_SD.3 (MOSI_CMD), R_SDMOSI.2, U1.34 (IO41)
- new net SD_SCLK: J_SD.5 (SCLK), R_SDSCLK.2, U1.33 (IO40)
- new net STATUS_LED_A: D_STATUS.2 (A), R_STATUS.2
- new net STATUS_LED_CTL: R_STATUS.1, U1.28 (IO35)
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Other:
- company: (none) -> Automatrix Engineering
- title: (none) -> Automatrix ESP32 PV-DG Controller

Commit message: hw: persist KiCad 10 validated Rev-A sources
Parts:
- removed C3_BOOT, C3_IN2, C_BOOT1: 0.1uF 50V, Capacitor_SMD:C_0603_1608Metric, symbol Automatrix:C
- removed C3_FB: 100pF, Capacitor_SMD:C_0603_1608Metric, symbol Automatrix:C
- removed C3_IN1: 10uF 35V, Capacitor_SMD:C_1206_3216Metric, symbol Automatrix:C_BIG
- removed C3_OUT1, C3_OUT2: 22uF 25V, Capacitor_SMD:C_1206_3216Metric, symbol Automatrix:C_BIG
- removed CINB: 100uF 50V, Capacitor_THT:CP_Radial_D10.0mm_P5.00mm, symbol Automatrix:C_BIG
- removed C_1V2: 10nF, Capacitor_SMD:C_0603_1608Metric, symbol Automatrix:C
- removed C_COMP: 6.8nF, Capacitor_SMD:C_0603_1608Metric, symbol Automatrix:C
- removed C_COMP_HF: 39pF, Capacitor_SMD:C_0603_1608Metric, symbol Automatrix:C
- removed C_EN: 1uF, Capacitor_SMD:C_0603_1608Metric, symbol Automatrix:C
- removed C_MCU1, C_SD1: 10uF, Capacitor_SMD:C_0805_2012Metric, symbol Automatrix:C_BIG
- removed C_MCU2, C_SD2: 0.1uF, Capacitor_SMD:C_0603_1608Metric, symbol Automatrix:C
- removed C_RS2321, C_RS2322, C_RS2323, C_RS2324, C_RS2325: 0.1uF DNP, Capacitor_SMD:C_0603_1608Metric, symbol Automatrix:CAP
- removed C_TOCAP: 4.7uF, Capacitor_SMD:C_0805_2012Metric, symbol Automatrix:C_BIG
- removed C_XI, C_XO: 18pF, Capacitor_SMD:C_0603_1608Metric, symbol Automatrix:C
- removed DZREV: 12V gate clamp, Diode_SMD:D_SOD-123, symbol Automatrix:ZENER
- removed D_DI1, D_DI2, D_DI3, D_DI4: 1N4148 reverse, Diode_SMD:D_SOD-123, symbol Automatrix:DIODE
- removed D_FLY1, D_FLY2, D_FLY3, D_FLY4: SS14, Diode_SMD:D_SMA, symbol Automatrix:DIODE
- removed D_LED1: RELAY1, LED_SMD:LED_0805_2012Metric, symbol Automatrix:LED
- removed D_LED2: RELAY2, LED_SMD:LED_0805_2012Metric, symbol Automatrix:LED
- removed D_LED3: RELAY3, LED_SMD:LED_0805_2012Metric, symbol Automatrix:LED
- removed D_LED4: RELAY4, LED_SMD:LED_0805_2012Metric, symbol Automatrix:LED
- removed D_OR_FIELD, D_OR_USB: SS34, Diode_SMD:D_SMA, symbol Automatrix:DIODE
- removed D_RS485A_TVS, D_RS485B_TVS: SM712, Package_TO_SOT_SMD:SOT-23, symbol Automatrix:TVS
- removed D_RTC_BAT, D_RTC_MAIN: BAT54, Diode_SMD:D_SOD-323, symbol Automatrix:DIODE
- removed D_STATUS: STATUS, LED_SMD:LED_0805_2012Metric, symbol Automatrix:LED
- removed D_USB_DN, D_USB_DP: USB ESD, Package_TO_SOT_SMD:SOT-23, symbol Automatrix:TVS
- removed F_HMI: 1.1A PTC, Fuse:Fuse_1206_3216Metric, symbol Automatrix:FUSE
- removed J_DI: DI1-4/COM, TerminalBlock_CUI:TerminalBlock_CUI_TB007-508-05_1x05_P5.08mm_Horizontal, symbol Automatrix:CONN5
- removed J_ETH: J1B1211CCD, Connector_RJ:RJ45_Cetus_J1B1211CCD_Horizontal, symbol Automatrix:MAGJACK
- removed J_HMI: HMI +5/GND/TX/RX, Connector_JST:JST_XH_B4B-XH-A_1x04_P2.50mm_Vertical, symbol Automatrix:CONN4
- removed J_PWR: 12/24V FIELD IN, TerminalBlock_CUI:TerminalBlock_CUI_TB007-508-02_1x02_P5.08mm_Horizontal, symbol Automatrix:CONN2
- removed J_RLY1: Relay1 NC/COM/NO, TerminalBlock_CUI:TerminalBlock_CUI_TB007-508-03_1x03_P5.08mm_Horizontal, symbol Automatrix:CONN3
- removed J_RLY2: Relay2 NC/COM/NO, TerminalBlock_CUI:TerminalBlock_CUI_TB007-508-03_1x03_P5.08mm_Horizontal, symbol Automatrix:CONN3
- removed J_RLY3: Relay3 NC/COM/NO, TerminalBlock_CUI:TerminalBlock_CUI_TB007-508-03_1x03_P5.08mm_Horizontal, symbol Automatrix:CONN3
- removed J_RLY4: Relay4 NC/COM/NO, TerminalBlock_CUI:TerminalBlock_CUI_TB007-508-03_1x03_P5.08mm_Horizontal, symbol Automatrix:CONN3
- removed J_RS232: RS232 GND/TX/RX DNP, Connector_JST:JST_XH_B3B-XH-A_1x03_P2.50mm_Vertical, symbol Automatrix:CONN3
- removed J_RS485A: RS485A A/B/GND, TerminalBlock_CUI:TerminalBlock_CUI_TB007-508-03_1x03_P5.08mm_Horizontal, symbol Automatrix:CONN3
- removed J_RS485B: RS485B A/B/GND, TerminalBlock_CUI:TerminalBlock_CUI_TB007-508-03_1x03_P5.08mm_Horizontal, symbol Automatrix:CONN3
- removed J_SD: microSD DNP, Connector_Card:microSD_HC_Hirose_DM3AT-SF-PEJM5, symbol Automatrix:SD
- removed J_USB: USB-C SERVICE, Connector_USB:USB_C_Receptacle_GCT_USB4105-xx-A_16P_TopMnt_Horizontal, symbol Automatrix:USB_C
- removed QREV: DMP6023LSS, Package_SO:SO-8_3.9x4.9mm_P1.27mm, symbol Automatrix:PMOS
- removed RREV, R_PD1, R_PD2, R_PD3, R_PD4: 100k, Resistor_SMD:R_0603_1608Metric, symbol Automatrix:R
- removed R_BOOT, R_DIPU1, R_DIPU2, R_DIPU3, R_DIPU4, R_EN, R_HMIRX_TOP, R_PM0, R_PM1, R_PM2, R_RS485A_DE, R_RS485B_DE, R_SDCS, R_SDMISO, R_SDMOSI, R_SDSCLK: 10k, Resistor_SMD:R_0603_1608Metric, symbol Automatrix:R
- removed R_CC1, R_CC2: 5.1k, Resistor_SMD:R_0603_1608Metric, symbol Automatrix:R
- removed R_COMP: 13k, Resistor_SMD:R_0603_1608Metric, symbol Automatrix:R
- removed R_DI1, R_DI2, R_DI3, R_DI4: 3.3k 0.25W, Resistor_SMD:R_1206_3216Metric, symbol Automatrix:R
- removed R_EN1: 523k, Resistor_SMD:R_0603_1608Metric, symbol Automatrix:R
- removed R_EN2: 84.5k, Resistor_SMD:R_0603_1608Metric, symbol Automatrix:R
- removed R_EXRES: 12.4k 1%, Resistor_SMD:R_0603_1608Metric, symbol Automatrix:R
- removed R_FB1: 53.6k, Resistor_SMD:R_0603_1608Metric, symbol Automatrix:R
- removed R_FB2: 10.2k, Resistor_SMD:R_0603_1608Metric, symbol Automatrix:R
- removed R_G1, R_G2, R_G3, R_G4, R_HMITX: 100R, Resistor_SMD:R_0603_1608Metric, symbol Automatrix:R
- removed R_HMIRX_BOT: 20k, Resistor_SMD:R_0603_1608Metric, symbol Automatrix:R
- removed R_LED1, R_LED2, R_LED3, R_LED4, R_STATUS: 1k, Resistor_SMD:R_0603_1608Metric, symbol Automatrix:R
- removed R_RS485A_BIASA, R_RS485A_BIASB, R_RS485B_BIASA, R_RS485B_BIASB: 680R DNP, Resistor_SMD:R_0603_1608Metric, symbol Automatrix:R
- removed R_RS485A_TERM, R_RS485B_TERM: 120R DNP, Resistor_SMD:R_1206_3216Metric, symbol Automatrix:R
- removed R_RT: 162k, Resistor_SMD:R_0603_1608Metric, symbol Automatrix:R
- removed R_SCL, R_SDA: 4.7k, Resistor_SMD:R_0603_1608Metric, symbol Automatrix:R
- removed R_XTAL: 1M, Resistor_SMD:R_0603_1608Metric, symbol Automatrix:R
- removed SW_BOOT: BOOT, Button_Switch_SMD:Panasonic_EVQPUJ_EVQPUA, symbol Automatrix:SW
- removed SW_RESET: RESET, Button_Switch_SMD:Panasonic_EVQPUJ_EVQPUA, symbol Automatrix:SW
- removed U_DI1, U_DI2, U_DI3, U_DI4: LTV-817, Package_DIP:DIP-4_W7.62mm, symbol Automatrix:OPTO
- removed U_RTC: PCF8563T DNP, Package_SO:SOIC-8_3.9x4.9mm_P1.27mm, symbol Automatrix:PCF8563
- removed Y_RTC: 32.768kHz, Crystal:Crystal_SMD_3215-2Pin_3.2x1.5mm, symbol Automatrix:CRYSTAL2
- added C1, C4, C6: 0.1uF 50V, Capacitor_SMD:C_0603_1608Metric, symbol Automatrix:C
- added C10: 1uF, Capacitor_SMD:C_0603_1608Metric, symbol Automatrix:C
- added C11, C17: 10uF, Capacitor_SMD:C_0805_2012Metric, symbol Automatrix:C_BIG
- added C12, C18: 0.1uF, Capacitor_SMD:C_0603_1608Metric, symbol Automatrix:C
- added C13: 4.7uF, Capacitor_SMD:C_0805_2012Metric, symbol Automatrix:C_BIG
- added C14: 10nF, Capacitor_SMD:C_0603_1608Metric, symbol Automatrix:C
- added C15, C16: 18pF, Capacitor_SMD:C_0603_1608Metric, symbol Automatrix:C
- added C19, C20, C21, C22, C23: 0.1uF DNP, Capacitor_SMD:C_0603_1608Metric, symbol Automatrix:CAP
- added C2: 6.8nF, Capacitor_SMD:C_0603_1608Metric, symbol Automatrix:C
- added C3: 39pF, Capacitor_SMD:C_0603_1608Metric, symbol Automatrix:C
- added C5: 10uF 35V, Capacitor_SMD:C_1206_3216Metric, symbol Automatrix:C_BIG
- added C7, C8: 22uF 25V, Capacitor_SMD:C_1206_3216Metric, symbol Automatrix:C_BIG
- added C9: 100pF, Capacitor_SMD:C_0603_1608Metric, symbol Automatrix:C
- added CINB1: 100uF 50V, Capacitor_THT:CP_Radial_D10.0mm_P5.00mm, symbol Automatrix:C_BIG
- added D1, D2: USB ESD, Package_TO_SOT_SMD:SOT-23, symbol Automatrix:TVS
- added D10, D12, D14, D8: SS14, Diode_SMD:D_SMA, symbol Automatrix:DIODE
- added D11: RELAY2, LED_SMD:LED_0805_2012Metric, symbol Automatrix:LED
- added D13: RELAY3, LED_SMD:LED_0805_2012Metric, symbol Automatrix:LED
- added D15: RELAY4, LED_SMD:LED_0805_2012Metric, symbol Automatrix:LED
- added D16, D17, D18, D19: 1N4148 reverse, Diode_SMD:D_SOD-123, symbol Automatrix:DIODE
- added D20, D21: BAT54, Diode_SMD:D_SOD-323, symbol Automatrix:DIODE
- added D3, D4: SS34, Diode_SMD:D_SMA, symbol Automatrix:DIODE
- added D5: STATUS, LED_SMD:LED_0805_2012Metric, symbol Automatrix:LED
- added D6, D7: SM712, Package_TO_SOT_SMD:SOT-23, symbol Automatrix:TVS
- added D9: RELAY1, LED_SMD:LED_0805_2012Metric, symbol Automatrix:LED
- added DZREV1: 12V gate clamp, Diode_SMD:D_SOD-123, symbol Automatrix:ZENER
- added F2: 1.1A PTC, Fuse:Fuse_1206_3216Metric, symbol Automatrix:FUSE
- added J1: 12/24V FIELD IN, TerminalBlock_CUI:TerminalBlock_CUI_TB007-508-02_1x02_P5.08mm_Horizontal, symbol Automatrix:CONN2
- added J10: Relay4 NC/COM/NO, TerminalBlock_CUI:TerminalBlock_CUI_TB007-508-03_1x03_P5.08mm_Horizontal, symbol Automatrix:CONN3
- added J11: DI1-4/COM, TerminalBlock_CUI:TerminalBlock_CUI_TB007-508-05_1x05_P5.08mm_Horizontal, symbol Automatrix:CONN5
- added J12: microSD DNP, Connector_Card:microSD_HC_Hirose_DM3AT-SF-PEJM5, symbol Automatrix:SD
- added J13: RS232 GND/TX/RX DNP, Connector_JST:JST_XH_B3B-XH-A_1x03_P2.50mm_Vertical, symbol Automatrix:CONN3
- added J2: USB-C SERVICE, Connector_USB:USB_C_Receptacle_GCT_USB4105-xx-A_16P_TopMnt_Horizontal, symbol Automatrix:USB_C
- added J3: J1B1211CCD, Connector_RJ:RJ45_Cetus_J1B1211CCD_Horizontal, symbol Automatrix:MAGJACK
- added J4: RS485A A/B/GND, TerminalBlock_CUI:TerminalBlock_CUI_TB007-508-03_1x03_P5.08mm_Horizontal, symbol Automatrix:CONN3
- added J5: RS485B A/B/GND, TerminalBlock_CUI:TerminalBlock_CUI_TB007-508-03_1x03_P5.08mm_Horizontal, symbol Automatrix:CONN3
- added J6: HMI +5/GND/TX/RX, Connector_JST:JST_XH_B4B-XH-A_1x04_P2.50mm_Vertical, symbol Automatrix:CONN4
- added J7: Relay1 NC/COM/NO, TerminalBlock_CUI:TerminalBlock_CUI_TB007-508-03_1x03_P5.08mm_Horizontal, symbol Automatrix:CONN3
- added J8: Relay2 NC/COM/NO, TerminalBlock_CUI:TerminalBlock_CUI_TB007-508-03_1x03_P5.08mm_Horizontal, symbol Automatrix:CONN3
- added J9: Relay3 NC/COM/NO, TerminalBlock_CUI:TerminalBlock_CUI_TB007-508-03_1x03_P5.08mm_Horizontal, symbol Automatrix:CONN3
- added QREV1: DMP6023LSS, Package_SO:SO-8_3.9x4.9mm_P1.27mm, symbol Automatrix:PMOS
- added R1: 523k, Resistor_SMD:R_0603_1608Metric, symbol Automatrix:R
- added R10, R14, R15, R16, R17, R21, R26, R41, R43, R45, R47, R50, R51, R52, R53, R9: 10k, Resistor_SMD:R_0603_1608Metric, symbol Automatrix:R
- added R11, R30, R33, R36, R39: 1k, Resistor_SMD:R_0603_1608Metric, symbol Automatrix:R
- added R12: 12.4k 1%, Resistor_SMD:R_0603_1608Metric, symbol Automatrix:R
- added R13: 1M, Resistor_SMD:R_0603_1608Metric, symbol Automatrix:R
- added R18, R22: 120R DNP, Resistor_SMD:R_1206_3216Metric, symbol Automatrix:R
- added R19, R20, R23, R24: 680R DNP, Resistor_SMD:R_0603_1608Metric, symbol Automatrix:R
- added R2: 84.5k, Resistor_SMD:R_0603_1608Metric, symbol Automatrix:R
- added R25, R28, R31, R34, R37: 100R, Resistor_SMD:R_0603_1608Metric, symbol Automatrix:R
- added R27: 20k, Resistor_SMD:R_0603_1608Metric, symbol Automatrix:R
- added R29, R32, R35, R38, RREV1: 100k, Resistor_SMD:R_0603_1608Metric, symbol Automatrix:R
- added R3: 162k, Resistor_SMD:R_0603_1608Metric, symbol Automatrix:R
- added R4: 53.6k, Resistor_SMD:R_0603_1608Metric, symbol Automatrix:R
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Connections:
- net 3V3: now also C11.1 (+), C12.1, C17.1 (+), C18.1, C23.1, C7.1 (+), C8.1 (+), C9.1, D20.2 (A), J12.4 (VDD), J3.10 (CT_TX), J3.11 (CT_RX)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
- net 5V_FIELD: now also D10.1 (K), D12.1 (K), D14.1 (K), D3.2 (A), D8.1 (K), F2.1, R30.1, R33.1, R36.1, R39.1, R4.1
- net 5V_HMI: now also F2.2, J6.1 (Pin_1)
- net 5V_LOGIC_IN: now also C5.1 (+), C6.1, D3.1 (K), D4.1 (K)
- net BUCK3_BST: now also C4.1
- net BUCK3_SW: now also C4.2
- net BUCK_BOOT: now also C1.1
- net BUCK_COMP: now also C3.1, R6.1
- net BUCK_COMP_RC: now also C2.1, R6.2
- net BUCK_EN: now also R1.2, R2.1
- net BUCK_FB: now also R4.2, R5.1
- net BUCK_RT: now also R3.1
- net BUCK_SW: now also C1.2
- net CHASSIS: now also J2.SH (SHIELD), J3.12 (CHASSIS), J3.9 (SHIELD)
- net DI1_FIELD: now also J11.1 (Pin_1), R40.1
- net DI1_LEDK: now also D16.1 (K), R40.2, U8.1 (A)
- net DI1_LOGIC: now also R41.2, U8.4 (C)
- net DI2_FIELD: now also J11.2 (Pin_2), R42.1
- net DI2_LEDK: now also D17.1 (K), R42.2, U9.1 (A)
- net DI2_LOGIC: now also R43.2, U9.4 (C)
- net DI3_FIELD: now also J11.3 (Pin_3), R44.1
- net DI3_LEDK: now also D18.1 (K), R44.2, U10.1 (A)
- net DI3_LOGIC: now also R45.2, U10.4 (C)
- net DI4_FIELD: now also J11.4 (Pin_4), R46.1
- net DI4_LEDK: now also D19.1 (K), R46.2, U11.1 (A)
- net DI4_LOGIC: now also R47.2, U11.4 (C)
- net DI_COM: now also D16.2 (A), D17.2 (A), D18.2 (A), D19.2 (A), J11.5 (Pin_5), U10.2 (K), U11.2 (K), U8.2 (K), U9.2 (K)
- net ESP_BOOT: now also R10.2, SW2.1
- net ESP_EN: now also C10.1, R9.2, SW1.1
- net ETH_1V2: now also C14.1
- net ETH_EXRES: now also R12.1
- net ETH_LED_ACT: now also J3.7 (LED_ACT_K)
- net ETH_LED_LINK: now also J3.5 (LED_LINK_K)
- net ETH_PMODE0: now also R16.2
- net ETH_PMODE1: now also R15.2
- net ETH_PMODE2: now also R14.2
- net ETH_RXN: now also J3.4 (PHY_RXN)
- net ETH_RXP: now also J3.3 (PHY_RXP)
- net ETH_TOCAP: now also C13.1 (+)
- net ETH_TXN: now also J3.2 (PHY_TXN)
- net ETH_TXP: now also J3.1 (PHY_TXP)
- net ETH_XI: now also C15.1, R13.1
- net ETH_XO: now also C16.1, R13.2
- net GND: now also C10.2, C11.2 (-), C12.2, C13.2 (-), C14.2, C15.2, C16.2, C17.2 (-), C18.2, C2.2, C21.2, C22.2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
- net HMI_RS232_RX: now also J13.3 (Pin_3)
- net HMI_RS232_TX: now also J13.2 (Pin_2)
- net HMI_RX: now also R26.2, R27.1
- net HMI_RX_IN: now also J6.4 (Pin_4), R26.1
- net HMI_TX: now also R25.1
- net HMI_TX_OUT: now also J6.3 (Pin_3), R25.2
- net RELAY1_COIL: now also D8.2 (A), D9.1 (K)
- net RELAY1_CTL: now also R28.1
- net RELAY1_GATE: now also R28.2, R29.1
- net RELAY2_COIL: now also D10.2 (A), D11.1 (K)
- net RELAY2_CTL: now also R31.1
- net RELAY2_GATE: now also R31.2, R32.1
- net RELAY3_COIL: now also D12.2 (A), D13.1 (K)
- net RELAY3_CTL: now also R34.1
- net RELAY3_GATE: now also R34.2, R35.1
- net RELAY4_COIL: now also D14.2 (A), D15.1 (K)
- net RELAY4_CTL: now also R37.1
- net RELAY4_GATE: now also R37.2, R38.1
- net REV_GATE: now also DZREV1.2 (A), QREV1.1 (G), RREV1.1
- net RLY1_COM: now also J7.2 (Pin_2)
- net RLY1_LED_A: now also D9.2 (A), R30.2
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
Commit message: pcb: freeze routed Rev-A H2 SI checkpoint [skip ci]
Parts:
- added C24, C25: 0.1uF DNP, Capacitor_SMD:C_0603_1608Metric, symbol Automatrix:CAP
- added C26, C27, C28, C29, C30, C31: 0.1uF, Capacitor_SMD:C_0603_1608Metric, symbol Automatrix:C
- added C32: 10uF 10V, Capacitor_SMD:C_0805_2012Metric, symbol Automatrix:C
- added C33: 22nF, Capacitor_SMD:C_0603_1608Metric, symbol Automatrix:C
- added C34: 6.8nF, Capacitor_SMD:C_0603_1608Metric, symbol Automatrix:C
- added C35: 1nF 2kV, Resistor_SMD:R_0805_2012Metric, symbol Automatrix:C
- added C36, C37: 0.1uF, Capacitor_SMD:C_0603_1608Metric, symbol Automatrix:CAP
- added D22, D24: AMBER 150080AS75000, LED_SMD:LED_0805_2012Metric, symbol Automatrix:LED0805_DIAG
- added D23, D25: GREEN 150080VS75000, LED_SMD:LED_0805_2012Metric, symbol Automatrix:LED0805_DIAG
- added D26: BRIGHT GREEN 150080VS75000, LED_SMD:LED_0805_2012Metric, symbol Automatrix:LED0805_DIAG
- added D27: RED 150080RS75000, LED_SMD:LED_0805_2012Metric, symbol Automatrix:LED0805_DIAG
- added FB1: 600R@100MHz >=1A, Resistor_SMD:R_0805_2012Metric, symbol Automatrix:FB
- added R54, R55, R56: 0R, Resistor_SMD:R_0603_1608Metric, symbol Automatrix:RES
- added R57, R58, R59, R60: 49.9R 1%, Resistor_SMD:R_0603_1608Metric, symbol Automatrix:RES
- added R61: 10R 1%, Resistor_SMD:R_0603_1608Metric, symbol Automatrix:RES
- added R62, R63: 330R, Resistor_SMD:R_0603_1608Metric, symbol Automatrix:RES
- added R64, R65, R66, R67, R70, R71: 680R, Resistor_SMD:R_0603_1608Metric, symbol Automatrix:RES
- added R68, R69: 100k, Resistor_SMD:R_0603_1608Metric, symbol Automatrix:RES
- added U13: SN74LVC1G17DBVR, Package_TO_SOT_SMD:SOT-23-5, symbol Automatrix:LVC1G17
- added U14: SN74LVC14APWR, Package_SO:TSSOP-14_4.4x5mm_P0.65mm, symbol Automatrix:LVC14
- C19, C20: value 0.1uF DNP -> 22pF DNP
- CIN1, CIN2: value 2.2uF 100V -> Murata GRM32ER72A225KA35L 2.2uF 100V X7R
- COUT1, COUT2: value 47uF 10V -> Murata GRM32ER61A476KE20L 47uF 10V X5R
- D1, D2: value USB ESD -> TPD1E05U06DYAR; footprint Package_TO_SOT_SMD:SOT-23 -> Diode_SMD:D_SOD-523; symbol Automatrix:TVS -> Automatrix:ESD1_UNI
- D10: value SS14 -> RELAY2; footprint Diode_SMD:D_SMA -> LED_SMD:LED_0805_2012Metric; symbol Automatrix:DIODE -> Automatrix:LED
- D11: value RELAY2 -> SS14; footprint LED_SMD:LED_0805_2012Metric -> Diode_SMD:D_SMA; symbol Automatrix:LED -> Automatrix:DIODE
- D12: value SS14 -> RELAY3; footprint Diode_SMD:D_SMA -> LED_SMD:LED_0805_2012Metric; symbol Automatrix:DIODE -> Automatrix:LED
- D13: value RELAY3 -> SS14; footprint LED_SMD:LED_0805_2012Metric -> Diode_SMD:D_SMA; symbol Automatrix:LED -> Automatrix:DIODE
- D14: value SS14 -> RELAY4; footprint Diode_SMD:D_SMA -> LED_SMD:LED_0805_2012Metric; symbol Automatrix:DIODE -> Automatrix:LED
- D15: value RELAY4 -> 1N4148 reverse; footprint LED_SMD:LED_0805_2012Metric -> Diode_SMD:D_SOD-123; symbol Automatrix:LED -> Automatrix:DIODE; now not fitted
- D19: value 1N4148 reverse -> BAT54; footprint Diode_SMD:D_SOD-123 -> Diode_SMD:D_SOD-323
- D21: value BAT54 -> TPD1E10B06DYAR; footprint Diode_SMD:D_SOD-323 -> Diode_SMD:D_SOD-523; symbol Automatrix:DIODE -> Automatrix:ESD1_BI; now fitted
- D5: value STATUS -> SM712; footprint LED_SMD:LED_0805_2012Metric -> Package_TO_SOT_SMD:SOT-23; symbol Automatrix:LED -> Automatrix:TVS
- D7: value SM712 -> SS14; footprint Package_TO_SOT_SMD:SOT-23 -> Diode_SMD:D_SMA; symbol Automatrix:TVS -> Automatrix:DIODE
- D8: value SS14 -> RELAY1; footprint Diode_SMD:D_SMA -> LED_SMD:LED_0805_2012Metric; symbol Automatrix:DIODE -> Automatrix:LED
- D9: value RELAY1 -> SS14; footprint LED_SMD:LED_0805_2012Metric -> Diode_SMD:D_SMA; symbol Automatrix:LED -> Automatrix:DIODE
- J1: value 12/24V FIELD IN -> Same Sky TB007-508-02BE
- J10: value Relay4 NC/COM/NO -> Phoenix MKDS 3/3-5.08 BK 1712193; footprint TerminalBlock_CUI:TerminalBlock_CUI_TB007-508-03_1x03_P5.08mm_Horizontal -> TerminalBlock_Phoenix:TerminalBlock_Phoenix_MKDS-3-3-5.08_1x03_P5.08mm_Horizontal
- J11: value DI1-4/COM -> Same Sky TB007-508-05BE DNP
- J2: value USB-C SERVICE -> GCT USB4105-GF-A-120
- J4: value RS485A A/B/GND -> Same Sky TB007-508-03BE
- J5: value RS485B A/B/GND -> Same Sky TB007-508-03BE
- J7: value Relay1 NC/COM/NO -> Phoenix MKDS 3/3-5.08 BK 1712193; footprint TerminalBlock_CUI:TerminalBlock_CUI_TB007-508-03_1x03_P5.08mm_Horizontal -> TerminalBlock_Phoenix:TerminalBlock_Phoenix_MKDS-3-3-5.08_1x03_P5.08mm_Horizontal
- J8: value Relay2 NC/COM/NO -> Phoenix MKDS 3/3-5.08 BK 1712193; footprint TerminalBlock_CUI:TerminalBlock_CUI_TB007-508-03_1x03_P5.08mm_Horizontal -> TerminalBlock_Phoenix:TerminalBlock_Phoenix_MKDS-3-3-5.08_1x03_P5.08mm_Horizontal
- J9: value Relay3 NC/COM/NO -> Phoenix MKDS 3/3-5.08 BK 1712193; footprint TerminalBlock_CUI:TerminalBlock_CUI_TB007-508-03_1x03_P5.08mm_Horizontal -> TerminalBlock_Phoenix:TerminalBlock_Phoenix_MKDS-3-3-5.08_1x03_P5.08mm_Horizontal
- L1: value 8.2uH >=5A -> Wurth 744393465082 8.2uH
- Q1, Q2, Q3, Q4: value AO3400A -> AOS AO3400A
- R11: value 1k -> 12.4k 1%
- R12: value 12.4k 1% -> 1M
- R13: value 1M -> 10k
- R17, R21: value 10k -> 120R DNP; footprint Resistor_SMD:R_0603_1608Metric -> Resistor_SMD:R_1206_3216Metric; now not fitted
- R18, R22: value 120R DNP -> 680R DNP; footprint Resistor_SMD:R_1206_3216Metric -> Resistor_SMD:R_0603_1608Metric
- R20: value 680R DNP -> 10k; now fitted
- R24: value 680R DNP -> 100R; now fitted
- R27: value 20k -> 1k
- R29, R32, R35: value 100k -> 10k
- R37: value 100R -> 3.3k 0.25W; footprint Resistor_SMD:R_0603_1608Metric -> Resistor_SMD:R_1206_3216Metric; now not fitted
- R38: value 100k -> 10k; now not fitted
- R39: value 1k -> 3.3k 0.25W; footprint Resistor_SMD:R_0603_1608Metric -> Resistor_SMD:R_1206_3216Metric; now not fitted
- R40, R42, R44: value 3.3k 0.25W -> 10k; footprint Resistor_SMD:R_1206_3216Metric -> Resistor_SMD:R_0603_1608Metric
- R41, R43: value 10k -> 3.3k 0.25W; footprint Resistor_SMD:R_0603_1608Metric -> Resistor_SMD:R_1206_3216Metric
- R45: value 10k -> 4.7k
- R46: value 3.3k 0.25W -> 4.7k; footprint Resistor_SMD:R_1206_3216Metric -> Resistor_SMD:R_0603_1608Metric
- R48, R49: value 4.7k -> 10k
- R51, R52: value 10k -> 27R; symbol Automatrix:R -> Automatrix:RES; now fitted
- R53: value 10k -> 0R; symbol Automatrix:R -> Automatrix:RES; now fitted
- Y1: value 25MHz -> Abracon ABM8-25.000MHZ-D2Y-T 25MHz
Connections:
- net 3V3: now also D19.2 (A), J3.12 (YLW+), R13.1, R18.1, R22.1, R38.1, R40.1, R42.1, R44.1, R46.1, C25.1, C36.1, C37.1, D26.2 (A), D27.2 (A), FB1.1, U13.5 (VCC), U14.14 (VCC); no longer C23.1, D20.2 (A), J3.11 (CT_RX), J3.6 (LED_LINK_A), J3.8 (LED_ACT_A), R16.1, R19.1, R23.1, R41.1, R43.1, R51.1, R52.1, R53.1, U2.11 (AVDD), U2.15 (AVDD), U2.17 (AVDD), U2.21 (AVDD), U2.4 (AVDD), U2.8 (AVDD)
- net 5V_FIELD: now also D11.1 (K), D13.1 (K), D7.1 (K), D9.1 (K), R27.1; no longer D10.1 (K), D12.1 (K), D14.1 (K), D8.1 (K), R39.1
- net CHASSIS: now also J3.13 (CH_GND), J3.8 (GHs_GND), C35.2; no longer J3.12 (CHASSIS), J3.9 (SHIELD)
- net DI1_FIELD: now also R37.1; no longer R40.1
- net DI1_LEDK: now also D15.1 (K), R37.2; no longer D16.1 (K), R40.2
- net DI1_LOGIC: now also R38.2; no longer R41.2
- net DI2_FIELD: now also R39.1; no longer R42.1
- net DI2_LEDK: now also D16.1 (K), R39.2; no longer D17.1 (K), R42.2
- net DI2_LOGIC: now also R40.2; no longer R43.2
- net DI3_FIELD: now also R41.1; no longer R44.1
- net DI3_LEDK: now also D17.1 (K), R41.2; no longer D18.1 (K), R44.2
- net DI3_LOGIC: now also R42.2; no longer R45.2
- net DI4_FIELD: now also R43.1; no longer R46.1
- net DI4_LEDK: now also D18.1 (K), R43.2; no longer D19.1 (K), R46.2
- net DI4_LOGIC: now also R44.2; no longer R47.2
- net DI_COM: now also D15.2 (A); no longer D19.2 (A)
- net ETH_EXRES: now also R11.1; no longer R12.1
- net ETH_LED_ACT: now also R63.1; no longer J3.7 (LED_ACT_K)
- net ETH_LED_LINK: now also R62.1; no longer J3.5 (LED_LINK_K)
- net ETH_PMODE0: now also R15.2; no longer R16.2
- net ETH_PMODE1: now also R14.2; no longer R15.2
- net ETH_PMODE2: now also R13.2; no longer R14.2
- net ETH_RXN: now also R56.1; no longer J3.4 (PHY_RXN)
- net ETH_RXP: now also R55.1; no longer J3.3 (PHY_RXP)
- net ETH_TXN: now also R54.1; no longer J3.2 (PHY_TXN)
- net ETH_TXP: now also R53.1; no longer J3.1 (PHY_TXP)
- net ETH_XI: now also R12.1; no longer R13.1
- net ETH_XO: now also R12.2; no longer R13.2
- net GND: now also C19.2, C20.2, D21.2 (GND), R11.2, R16.2, R19.2, R23.2, R26.2, C24.2, C25.2, C26.2, C27.2, C28.2, C29.2, C30.2, C31.2, C32.2, C33.2, C34.2, C35.1, C36.2, C37.2, D22.1 (K), D23.1 (K), D24.1 (K), D25.1 (K), R68.2, R69.2, U13.3 (GND), U14.7 (GND); no longer C21.2, C22.2, D5.1 (K), R12.2, R17.2, R21.2, R24.2, R27.2, R38.2
- net HMI_RX: now also U13.4 (Y); no longer R26.2, R27.1
- net HMI_RX_IN: now also D21.1 (IO), U13.2 (A); no longer R26.1
- net HMI_TX: now also R24.1; no longer R25.1
- net HMI_TX_OUT: now also R24.2; no longer R25.2
- net RELAY1_COIL: now also D7.2 (A), D8.1 (K); no longer D8.2 (A), D9.1 (K)
- net RELAY1_CTL: now also R25.1; no longer R28.1
- net RELAY1_GATE: now also R25.2, R26.1; no longer R28.2, R29.1
- net RELAY2_COIL: now also D10.1 (K), D9.2 (A); no longer D10.2 (A), D11.1 (K)
- net RELAY2_CTL: now also R28.1; no longer R31.1
- net RELAY2_GATE: now also R28.2, R29.1; no longer R31.2, R32.1
- net RELAY3_COIL: now also D11.2 (A), D12.1 (K); no longer D12.2 (A), D13.1 (K)
- net RELAY3_CTL: now also R31.1; no longer R34.1
- net RELAY3_GATE: now also R31.2, R32.1; no longer R34.2, R35.1
- net RELAY4_COIL: now also D13.2 (A), D14.1 (K); no longer D14.2 (A), D15.1 (K)
- net RELAY4_CTL: now also R34.1; no longer R37.1
- net RELAY4_GATE: now also R34.2, R35.1; no longer R37.2, R38.1
- net RLY1_LED_A: now also D8.2 (A), R27.2; no longer D9.2 (A), R30.2
- net RLY2_LED_A: now also D10.2 (A), R30.2; no longer D11.2 (A), R33.2
- net RLY3_LED_A: now also D12.2 (A), R33.2; no longer D13.2 (A), R36.2
- net RLY4_LED_A: now also D14.2 (A), R36.2; no longer D15.2 (A), R39.2
- net RS232_C1M: now also C21.2; no longer C19.2
- net RS232_C1P: now also C21.1; no longer C19.1
- net RS232_C2M: now also C22.2; no longer C20.2
- net RS232_C2P: now also C22.1; no longer C20.1
- net RS232_VMINUS: now also C24.1; no longer C22.1
- net RS232_VPLUS: now also C23.1; no longer C21.1
- net RS485A_A: now also D5.1 (A), R17.1, R18.2; no longer D6.1 (A), R18.1, R19.2
- net RS485A_B: now also D5.2 (K), R17.2, R19.1; no longer D6.2 (K), R18.2, R20.1
- net RS485A_DE: now also R16.1; no longer R17.1
- net RS485A_RX: now also U14.3 (2A)
- net RS485A_TX: now also U14.1 (1A)
- net RS485B_A: now also D6.1 (A), R21.1, R22.2; no longer D7.1 (A), R22.1, R23.2
- net RS485B_B: now also D6.2 (K), R21.2, R23.1; no longer D7.2 (K), R22.2, R24.1
- net RS485B_DE: now also R20.1; no longer R21.1
- net RS485B_RX: now also U14.9 (4A)
- net RS485B_TX: now also U14.5 (3A)
- net RTC_BAT: now also D20.2 (A); no longer D21.2 (A)
- net RTC_SCL: now also R46.2; no longer R49.2
- net RTC_SDA: now also R45.2; no longer R48.2
- net RTC_VDD: now also D19.1 (K); no longer D21.1 (K)
- net SD_CS: now also R47.2; no longer R50.2
- net SD_MISO: now also R50.2; no longer R53.2
- net SD_MOSI: now also R48.2; no longer R51.2
- net SD_SCLK: now also R49.2; no longer R52.2
- net STATUS_LED_CTL: now also R68.1, U14.11 (5A); no longer R11.1
- net USB_D+: now also R52.2; no longer U1.14 (IO20)
- net USB_D-: now also R51.2; no longer U1.13 (IO19)
- net STATUS_ALERT_CTL: now reaches U1.23 (IO21)
- net STATUS_ALERT_CTL: now also R69.1, U14.13 (6A)
- removed net STATUS_LED_A: D5.2 (A), R11.2
- new net 3V3A: C26.1, C27.1, C28.1, C29.1, C30.1, C31.1, C32.1, FB1.2, R57.1, R58.1, R59.1, R60.1, R61.1, U2.11 (AVDD), U2.15 (AVDD), U2.17 (AVDD), U2.21 (AVDD), U2.4 (AVDD), U2.8 (AVDD)
- new net DIAG_A_RX_DRV: R65.1, U14.4 (2Y)
- new net DIAG_A_TX_DRV: R64.1, U14.2 (1Y)
- new net DIAG_B_RX_DRV: R67.1, U14.8 (4Y)
- new net DIAG_B_TX_DRV: R66.1, U14.6 (3Y)
- new net ETH_LED_ACT_K: J3.11 (YLW-), R63.2
- new net ETH_LED_LINK_K: J3.9 (GRN-), R62.2
- new net ETH_RCT: C34.1, J3.5 (RCT)
- new net ETH_RXN_MAG: J3.6 (RD-), R56.2, R60.2
- new net ETH_RXP_MAG: J3.4 (RD+), R55.2, R59.2
- new net ETH_TCT: C33.1, J3.2 (TCT), R61.2
- new net ETH_TXN_MAG: J3.3 (TD-), R54.2, R58.2
- new net ETH_TXP_MAG: J3.1 (TD+), R53.2, R57.2
- new net LED_A_RX_A: D23.2 (A), R65.2
- new net LED_A_TX_A: D22.2 (A), R64.2
- new net LED_B_RX_A: D25.2 (A), R67.2
- new net LED_B_TX_A: D24.2 (A), R66.2
- new net STATUS_GREEN_DRV: R70.1, U14.10 (5Y)
- new net STATUS_GREEN_K: D26.1 (K), R70.2
- new net STATUS_RED_DRV: R71.1, U14.12 (6Y)
- new net STATUS_RED_K: D27.1 (K), R71.2
- new net USB_D+_MCU: C20.1, R52.1, U1.14 (IO20)
- new net USB_D-_MCU: C19.1, R51.1, U1.13 (IO19)
- no-connect marks 27 -> 28
Other:
- moved on the sheet: BT1, C11, C12, C13, C14, C15, C16, C17, C18, C19, C20, C21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
