File: hardware/kicad/Automatrix_PVDG_RevA.kicad_pcb (KiCad board)
At the start: 4 copper layers, 145 x 95 mm, 153 parts, among them J1 12/24V FIELD IN, J10 Relay4 NC/COM/NO, J11 DI1-4/COM, J12 microSD DNP, J13 RS232 GND/TX/RX DNP, J2 USB-C SERVICE, J3 J1B1211CCD, J4 RS485A A/B/GND, J5 RS485B A/B/GND, J6 HMI +5/GND/TX/RX, J7 Relay1 NC/COM/NO, J8 Relay2 NC/COM/NO, J9 Relay3 NC/COM/NO, K1 HF3FF/005-1ZST, K2 HF3FF/005-1ZST, K3 HF3FF/005-1ZST, K4 HF3FF/005-1ZST, Q1 AO3400A, Q2 AO3400A, Q3 AO3400A, Q4 AO3400A, SW1 RESET, SW2 BOOT, U1 ESP32-S3-WROOM-1-N8, U10 LTV-817, U11 LTV-817, U12 PCF8563T DNP, U2 W5500, U3 THVD1410D, U4 THVD1410D, U5 TPS54360B, U6 AP63203WU-7, U7 MAX3232 DNP, U8 LTV-817, U9 LTV-817, Y1 25MHz, Y2 32.768kHz

Commit message: pcb: freeze routed Rev-A H2 [skip ci]
Routing:
- net GND: track 0.00 -> 833.1 mm, vias 0 -> 9
- net 3V3: track 0.00 -> 501.4 mm, vias 0 -> 10
- net 5V_FIELD: track 0.00 -> 318.9 mm, vias 0 -> 6
- net 5V_LOGIC_IN: track 0.00 -> 186.7 mm, vias 0 -> 4
- net DI4_LOGIC: track 0.00 -> 163.5 mm, vias 0 -> 2
- net USB_D-: track 0.00 -> 151.6 mm, vias 0 -> 2
- net DI3_LOGIC: track 0.00 -> 151.3 mm, vias 0 -> 2
- net RELAY4_CTL: track 0.00 -> 150.1 mm, vias 0 -> 3
- net USB_D+: track 0.00 -> 147.3 mm, vias 0 -> 3
- net DI2_LOGIC: track 0.00 -> 144.7 mm, vias 0 -> 2
- net BUCK_COMP: track 0.00 -> 137.5 mm, vias 0 -> 3
- net SD_MOSI: track 0.00 -> 131.6 mm, vias 0 -> 2
- net RELAY3_CTL: track 0.00 -> 126.9 mm, vias 0 -> 3
- net DI1_LOGIC: track 0.00 -> 116.8 mm, vias 0 -> 2
- net SD_CS: track 0.00 -> 114.7 mm, vias 0 -> 3
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
Commit message: pcb: freeze routed Rev-A H2 [skip ci]
Routing:
- net BUCK_COMP: track 137.5 -> 101.7 mm
- net VIN_PROTECTED: track 69.1 -> 87.5 mm
- net GND: track 833.1 -> 818.2 mm, vias 9 -> 10
- net RS485A_A: track 52.3 -> 38.3 mm, vias 2 -> 0
- net DI3_LOGIC: track 151.3 -> 138.4 mm, vias 2 -> 3
- net RS485A_B: track 55.7 -> 44.0 mm, vias 1 -> 2
- net 3V3: track 501.4 -> 512.8 mm, vias 10 -> 7
- net ETH_1V2: track 27.8 -> 16.5 mm
- net RLY1_LED_A: track 7.29 -> 18.4 mm
- net VIN_RAW: track 35.0 -> 45.0 mm
- net RTC_X2: track 12.6 -> 22.1 mm, vias 2 -> 0
- net USB_D+: track 147.3 -> 138.4 mm
- net 5V_LOGIC_IN: track 186.7 -> 178.1 mm
- net SD_SCLK: track 111.5 -> 119.3 mm, vias 2 -> 3
- net RELAY1_COIL: track 49.7 -> 42.3 mm, vias 2 -> 1
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
Commit message: pcb: freeze routed Rev-A H2 SI checkpoint [skip ci]
Parts:
- added C24: 0.1uF DNP, C_0603_1608Metric, F.Cu at (78.0, 76.0)
- added C25: 0.1uF DNP, C_0603_1608Metric, F.Cu at (90.0, 76.0)
- added C26: 0.1uF, C_0603_1608Metric, F.Cu at (102.0, 62.0)
- added C27: 0.1uF, C_0603_1608Metric, F.Cu at (102.0, 66.0)
- added C28: 0.1uF, C_0603_1608Metric, F.Cu at (107.0, 57.0)
- added C29: 0.1uF, C_0603_1608Metric, F.Cu at (107.0, 71.0)
- added C30: 0.1uF, C_0603_1608Metric, F.Cu at (103.0, 60.0)
- added C31: 0.1uF, C_0603_1608Metric, F.Cu at (103.0, 68.0)
- added C32: 10uF 10V, C_0805_2012Metric, F.Cu at (98.0, 64.0)
- added C33: 22nF, C_0603_1608Metric, F.Cu at (107.0, 73.0)
- added C34: 6.8nF, C_0603_1608Metric, F.Cu at (103.0, 58.0)
- added C35: 1nF 2kV, R_0805_2012Metric, F.Cu at (103.0, 71.0)
- added C36: 0.1uF, C_0603_1608Metric, F.Cu at (77.5, 89.5)
- added C37: 0.1uF, C_0603_1608Metric, F.Cu at (6.00, 71.0)
- added D22: AMBER 150080AS75000, LED_0805_2012Metric, F.Cu at (32.0, 78.0)
- added D23: GREEN 150080VS75000, LED_0805_2012Metric, F.Cu at (44.5, 74.5)
- added D24: AMBER 150080AS75000, LED_0805_2012Metric, F.Cu at (54.0, 78.0)
- added D25: GREEN 150080VS75000, LED_0805_2012Metric, F.Cu at (66.0, 78.0)
- added D26: BRIGHT GREEN 150080VS75000, LED_0805_2012Metric, F.Cu at (6.00, 40.0)
- added D27: RED 150080RS75000, LED_0805_2012Metric, F.Cu at (10.0, 43.0)
- added FB1: 600R@100MHz >=1A, R_0805_2012Metric, F.Cu at (98.0, 61.0)
- added R54: 0R, R_0603_1608Metric, F.Cu at (123.6, 68.5)
- added R55: 0R, R_0603_1608Metric, F.Cu at (123.6, 60.3)
- added R56: 0R, R_0603_1608Metric, F.Cu at (123.6, 62.8)
- added R57: 49.9R 1%, R_0603_1608Metric, F.Cu at (126.6, 66.8)
- added R58: 49.9R 1%, R_0603_1608Metric, F.Cu at (126.6, 70.2)
- added R59: 49.9R 1%, R_0603_1608Metric, F.Cu at (126.6, 59.5)
- added R60: 49.9R 1%, R_0603_1608Metric, F.Cu at (126.6, 63.0)
- added R61: 10R 1%, R_0603_1608Metric, F.Cu at (99.0, 58.0)
- added R62: 330R, R_0603_1608Metric, F.Cu at (94.0, 62.0)
- added R63: 330R, R_0603_1608Metric, F.Cu at (94.0, 66.0)
- added R64: 680R, R_0603_1608Metric, F.Cu at (49.0, 74.0)
- added R65: 680R, R_0603_1608Metric, F.Cu at (49.0, 72.0)
- added R66: 680R, R_0603_1608Metric, F.Cu at (54.0, 81.0)
- added R67: 680R, R_0603_1608Metric, F.Cu at (70.0, 78.0)
- added R68: 100k, R_0603_1608Metric, F.Cu at (17.0, 39.0)
- added R69: 100k, R_0603_1608Metric, F.Cu at (23.0, 44.0)
- added R70: 680R, R_0603_1608Metric, F.Cu at (3.00, 82.0)
- added R71: 680R, R_0603_1608Metric, F.Cu at (22.0, 42.0)
- added U13: SN74LVC1G17DBVR, SOT-23-5, F.Cu at (76.0, 83.5)
- added U14: SN74LVC14APWR, TSSOP-14_4.4x5mm_P0.65mm, F.Cu at (48.0, 48.0)
- C19, C20: value 0.1uF DNP -> 22pF DNP
- CIN1, CIN2: value 2.2uF 100V -> Murata GRM32ER72A225KA35L 2.2uF 100V X7R
- COUT1, COUT2: value 47uF 10V -> Murata GRM32ER61A476KE20L 47uF 10V X5R
- D1, D2: value USB ESD -> TPD1E05U06DYAR; footprint SOT-23 -> D_SOD-523
- D10: value SS14 -> RELAY2; footprint D_SMA -> LED_0805_2012Metric
- D11: value RELAY2 -> SS14; footprint LED_0805_2012Metric -> D_SMA
- D12: value SS14 -> RELAY3; footprint D_SMA -> LED_0805_2012Metric
- D13: value RELAY3 -> SS14; footprint LED_0805_2012Metric -> D_SMA
- D14: value SS14 -> RELAY4; footprint D_SMA -> LED_0805_2012Metric
- D15: value RELAY4 -> 1N4148 reverse; footprint LED_0805_2012Metric -> D_SOD-123
- D19: value 1N4148 reverse -> BAT54; footprint D_SOD-123 -> D_SOD-323
- D21: value BAT54 -> TPD1E10B06DYAR; footprint D_SOD-323 -> D_SOD-523
- D5: value STATUS -> SM712; footprint LED_0805_2012Metric -> SOT-23
- D7: value SM712 -> SS14; footprint SOT-23 -> D_SMA
- D8: value SS14 -> RELAY1; footprint D_SMA -> LED_0805_2012Metric
- D9: value RELAY1 -> SS14; footprint LED_0805_2012Metric -> D_SMA
- J1: value 12/24V FIELD IN -> Same Sky TB007-508-02BE
- J10: value Relay4 NC/COM/NO -> Phoenix MKDS 3/3-5.08 BK 1712193; footprint TerminalBlock_CUI_TB007-508-03_1x03_P5.08mm_Horizontal -> TerminalBlock_Phoenix_MKDS-3-3-5.08_1x03_P5.08mm_Horizontal
- J11: value DI1-4/COM -> Same Sky TB007-508-05BE DNP
- J2: value USB-C SERVICE -> GCT USB4105-GF-A-120
- J4: value RS485A A/B/GND -> Same Sky TB007-508-03BE
- J5: value RS485B A/B/GND -> Same Sky TB007-508-03BE
- J7: value Relay1 NC/COM/NO -> Phoenix MKDS 3/3-5.08 BK 1712193; footprint TerminalBlock_CUI_TB007-508-03_1x03_P5.08mm_Horizontal -> TerminalBlock_Phoenix_MKDS-3-3-5.08_1x03_P5.08mm_Horizontal
- J8: value Relay2 NC/COM/NO -> Phoenix MKDS 3/3-5.08 BK 1712193; footprint TerminalBlock_CUI_TB007-508-03_1x03_P5.08mm_Horizontal -> TerminalBlock_Phoenix_MKDS-3-3-5.08_1x03_P5.08mm_Horizontal
- J9: value Relay3 NC/COM/NO -> Phoenix MKDS 3/3-5.08 BK 1712193; footprint TerminalBlock_CUI_TB007-508-03_1x03_P5.08mm_Horizontal -> TerminalBlock_Phoenix_MKDS-3-3-5.08_1x03_P5.08mm_Horizontal
- L1: value 8.2uH >=5A -> Wurth 744393465082 8.2uH
- Q1, Q2, Q3, Q4: value AO3400A -> AOS AO3400A
- R11: value 1k -> 12.4k 1%
- R12: value 12.4k 1% -> 1M
- R13: value 1M -> 10k
- R17, R21: value 10k -> 120R DNP; footprint R_0603_1608Metric -> R_1206_3216Metric
- R18, R22: value 120R DNP -> 680R DNP; footprint R_1206_3216Metric -> R_0603_1608Metric
- R20: value 680R DNP -> 10k
- R24: value 680R DNP -> 100R
- R27: value 20k -> 1k
- R29, R32, R35, R38: value 100k -> 10k
- R37: value 100R -> 3.3k 0.25W; footprint R_0603_1608Metric -> R_1206_3216Metric
- R39: value 1k -> 3.3k 0.25W; footprint R_0603_1608Metric -> R_1206_3216Metric
- R40, R42, R44: value 3.3k 0.25W -> 10k; footprint R_1206_3216Metric -> R_0603_1608Metric
- R41, R43: value 10k -> 3.3k 0.25W; footprint R_0603_1608Metric -> R_1206_3216Metric
- R45: value 10k -> 4.7k
- R46: value 3.3k 0.25W -> 4.7k; footprint R_1206_3216Metric -> R_0603_1608Metric
- R48, R49: value 4.7k -> 10k
- R51, R52: value 10k -> 27R
- R53: value 10k -> 0R
- Y1: value 25MHz -> Abracon ABM8-25.000MHZ-D2Y-T 25MHz
- moved D4 130.1 mm to (6.50, 78.5)
- moved R43 123.6 mm to (123.0, 72.0)
- moved R51 111.1 mm to (23.5, 64.0)
- moved R46 109.7 mm to (23.0, 48.0)
- moved R45 107.1 mm to (131.0, 39.0)
- moved R44 104.4 mm to (14.0, 41.0)
- moved R38 94.4 mm to (14.0, 43.0)
- moved R40 92.1 mm to (4.00, 75.0)
- moved R50 90.4 mm to (18.0, 71.0)
- moved R27 89.7 mm to (13.0, 39.0)
- moved R26 87.7 mm to (17.0, 30.0)
- moved R42 84.8 mm to (23.0, 50.0)
- moved R48 83.5 mm to (23.0, 46.0)
- moved R52 83.0 mm to (23.5, 66.0)
- moved R25 82.5 mm to (17.0, 32.0)
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Connections:
- C19 pad 1: RS232_C1P -> USB_D-_MCU
- C19 pad 2: RS232_C1M -> GND
- C20 pad 1: RS232_C2P -> USB_D+_MCU
- C20 pad 2: RS232_C2M -> GND
- C21 pad 1: RS232_VPLUS -> RS232_C1P
- C21 pad 2: GND -> RS232_C1M
- C22 pad 1: RS232_VMINUS -> RS232_C2P
- C22 pad 2: GND -> RS232_C2M
- C23 pad 1: 3V3 -> RS232_VPLUS
- D10 pad 1: 5V_FIELD -> RELAY2_COIL
- D10 pad 2: RELAY2_COIL -> RLY2_LED_A
- D11 pad 1: RELAY2_COIL -> 5V_FIELD
- D11 pad 2: RLY2_LED_A -> RELAY3_COIL
- D12 pad 1: 5V_FIELD -> RELAY3_COIL
- D12 pad 2: RELAY3_COIL -> RLY3_LED_A
- D13 pad 1: RELAY3_COIL -> 5V_FIELD
- D13 pad 2: RLY3_LED_A -> RELAY4_COIL
- D14 pad 1: 5V_FIELD -> RELAY4_COIL
- D14 pad 2: RELAY4_COIL -> RLY4_LED_A
- D15 pad 1: RELAY4_COIL -> DI1_LEDK
- D15 pad 2: RLY4_LED_A -> DI_COM
- D16 pad 1: DI1_LEDK -> DI2_LEDK
- D17 pad 1: DI2_LEDK -> DI3_LEDK
- D18 pad 1: DI3_LEDK -> DI4_LEDK
- D19 pad 1: DI4_LEDK -> RTC_VDD
- D19 pad 2: DI_COM -> 3V3
- D20 pad 2: 3V3 -> RTC_BAT
- D21 pad 1: RTC_VDD -> HMI_RX_IN
- D21 pad 2: RTC_BAT -> GND
- D5 pad 1: GND -> RS485A_A
- D5 pad 2: STATUS_LED_A -> RS485A_B
- D6 pad 1: RS485A_A -> RS485B_A
- D6 pad 2: RS485A_B -> RS485B_B
- D7 pad 1: RS485B_A -> 5V_FIELD
- D7 pad 2: RS485B_B -> RELAY1_COIL
- D8 pad 1: 5V_FIELD -> RELAY1_COIL
- D8 pad 2: RELAY1_COIL -> RLY1_LED_A
- D9 pad 1: RELAY1_COIL -> 5V_FIELD
- D9 pad 2: RLY1_LED_A -> RELAY2_COIL
- J3 pad 1: ETH_TXP -> ETH_TXP_MAG
- J3 pad 11: 3V3 -> ETH_LED_ACT_K
- J3 pad 12: CHASSIS -> 3V3
- J3 pad 13: (no net) -> CHASSIS
- J3 pad 2: ETH_TXN -> ETH_TCT
- J3 pad 3: ETH_RXP -> ETH_TXN_MAG
- J3 pad 4: ETH_RXN -> ETH_RXP_MAG
- J3 pad 5: ETH_LED_LINK -> ETH_RCT
- J3 pad 6: 3V3 -> ETH_RXN_MAG
- J3 pad 7: ETH_LED_ACT -> (no net)
- J3 pad 8: 3V3 -> CHASSIS
- J3 pad 9: CHASSIS -> ETH_LED_LINK_K
- R11 pad 1: STATUS_LED_CTL -> ETH_EXRES
- R11 pad 2: STATUS_LED_A -> GND
- R12 pad 1: ETH_EXRES -> ETH_XI
- R12 pad 2: GND -> ETH_XO
- R13 pad 1: ETH_XI -> 3V3
- R13 pad 2: ETH_XO -> ETH_PMODE2
- R14 pad 2: ETH_PMODE2 -> ETH_PMODE1
- R15 pad 2: ETH_PMODE1 -> ETH_PMODE0
- R16 pad 1: 3V3 -> RS485A_DE
- R16 pad 2: ETH_PMODE0 -> GND
- R17 pad 1: RS485A_DE -> RS485A_A
- R17 pad 2: GND -> RS485A_B
- R18 pad 1: RS485A_A -> 3V3
- R18 pad 2: RS485A_B -> RS485A_A
- R19 pad 1: 3V3 -> RS485A_B
- R19 pad 2: RS485A_A -> GND
- R20 pad 1: RS485A_B -> RS485B_DE
- R21 pad 1: RS485B_DE -> RS485B_A
- R21 pad 2: GND -> RS485B_B
- R22 pad 1: RS485B_A -> 3V3
- R22 pad 2: RS485B_B -> RS485B_A
- R23 pad 1: 3V3 -> RS485B_B
- R23 pad 2: RS485B_A -> GND
- R24 pad 1: RS485B_B -> HMI_TX
- R24 pad 2: GND -> HMI_TX_OUT
- R25 pad 1: HMI_TX -> RELAY1_CTL
- R25 pad 2: HMI_TX_OUT -> RELAY1_GATE
- R26 pad 1: HMI_RX_IN -> RELAY1_GATE
- R26 pad 2: HMI_RX -> GND
- R27 pad 1: HMI_RX -> 5V_FIELD
- R27 pad 2: GND -> RLY1_LED_A
- R28 pad 1: RELAY1_CTL -> RELAY2_CTL
- R28 pad 2: RELAY1_GATE -> RELAY2_GATE
- R29 pad 1: RELAY1_GATE -> RELAY2_GATE
- R30 pad 2: RLY1_LED_A -> RLY2_LED_A
- R31 pad 1: RELAY2_CTL -> RELAY3_CTL
- R31 pad 2: RELAY2_GATE -> RELAY3_GATE
- R32 pad 1: RELAY2_GATE -> RELAY3_GATE
- R33 pad 2: RLY2_LED_A -> RLY3_LED_A
- R34 pad 1: RELAY3_CTL -> RELAY4_CTL
- R34 pad 2: RELAY3_GATE -> RELAY4_GATE
- R35 pad 1: RELAY3_GATE -> RELAY4_GATE
- R36 pad 2: RLY3_LED_A -> RLY4_LED_A
- R37 pad 1: RELAY4_CTL -> DI1_FIELD
- R37 pad 2: RELAY4_GATE -> DI1_LEDK
- R38 pad 1: RELAY4_GATE -> 3V3
- R38 pad 2: GND -> DI1_LOGIC
- R39 pad 1: 5V_FIELD -> DI2_FIELD
- R39 pad 2: RLY4_LED_A -> DI2_LEDK
- R40 pad 1: DI1_FIELD -> 3V3
- R40 pad 2: DI1_LEDK -> DI2_LOGIC
- R41 pad 1: 3V3 -> DI3_FIELD
- R41 pad 2: DI1_LOGIC -> DI3_LEDK
- R42 pad 1: DI2_FIELD -> 3V3
- R42 pad 2: DI2_LEDK -> DI3_LOGIC
- R43 pad 1: 3V3 -> DI4_FIELD
- R43 pad 2: DI2_LOGIC -> DI4_LEDK
- R44 pad 1: DI3_FIELD -> 3V3
- R44 pad 2: DI3_LEDK -> DI4_LOGIC
- R45 pad 2: DI3_LOGIC -> RTC_SDA
- R46 pad 1: DI4_FIELD -> 3V3
- R46 pad 2: DI4_LEDK -> RTC_SCL
- R47 pad 2: DI4_LOGIC -> SD_CS
- R48 pad 2: RTC_SDA -> SD_MOSI
- R49 pad 2: RTC_SCL -> SD_SCLK
- R50 pad 2: SD_CS -> SD_MISO
- R51 pad 1: 3V3 -> USB_D-_MCU
- R51 pad 2: SD_MOSI -> USB_D-
- R52 pad 1: 3V3 -> USB_D+_MCU
- R52 pad 2: SD_SCLK -> USB_D+
- R53 pad 1: 3V3 -> ETH_TXP
- R53 pad 2: SD_MISO -> ETH_TXP_MAG
- U1 pad 13: USB_D- -> USB_D-_MCU
- U1 pad 14: USB_D+ -> USB_D+_MCU
- U1 pad 23: (no net) -> STATUS_ALERT_CTL
- U2 pad 11: 3V3 -> 3V3A
- U2 pad 15: 3V3 -> 3V3A
- U2 pad 17: 3V3 -> 3V3A
- U2 pad 21: 3V3 -> 3V3A
- U2 pad 4: 3V3 -> 3V3A
- U2 pad 8: 3V3 -> 3V3A
Routing:
- net GND: track 818.2 -> 59.1 mm, vias 10 -> 41
- net USB_5V: track 11.3 -> 159.2 mm, vias 0 -> 4
- net 5V_LOGIC_IN: track 178.1 -> 62.6 mm, vias 4 -> 0
- net 3V3A: track 0.00 -> 90.3 mm, vias 0 -> 4
- net 3V3: track 512.8 -> 428.1 mm, vias 7 -> 8
- net STATUS_GREEN_DRV: track 0.00 -> 75.7 mm, vias 0 -> 5
- net BUCK_COMP: track 101.7 -> 27.0 mm, vias 3 -> 0
- net 5V_FIELD: track 316.0 -> 385.6 mm, vias 7 -> 8
- net ETH_LED_LINK_K: track 0.00 -> 62.5 mm, vias 0 -> 1
- net BUCK3_SW: track 70.8 -> 13.8 mm, vias 3 -> 0
- net ETH_LED_ACT_K: track 0.00 -> 54.5 mm, vias 0 -> 1
- net CHASSIS: track 31.2 -> 83.8 mm
- net ETH_TCT: track 0.00 -> 50.1 mm, vias 0 -> 2
- net RS232_C1M: track 50.3 -> 3.54 mm, vias 2 -> 0
- net STATUS_ALERT_CTL: track 0.00 -> 46.8 mm, vias 0 -> 2
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- added copper zone on B.Cu, net GND
- added copper zone on F.Cu, net GND
- added copper zone on In1.Cu, net GND

Commit message: pcb: freeze routed Rev-A H2 SI checkpoint [skip ci]
Parts:
- moved R70 43.4 mm to (22.0, 43.0)
- moved R10 36.1 mm to (4.00, 73.0)
- moved R9 33.5 mm to (10.0, 40.0)
- moved R40 33.5 mm to (14.0, 43.0)
- moved R68 32.0 mm to (18.0, 71.0)
- moved R42 31.4 mm to (4.00, 75.0)
- moved R50 30.0 mm to (18.0, 41.0)
- moved R48 11.4 mm to (14.0, 39.0)
- moved R27 10.6 mm to (21.0, 32.0)
- moved R38 10.0 mm to (6.00, 37.0)
- moved R49 9.22 mm to (24.0, 48.0)
- moved D26 5.00 mm to (10.0, 43.0)
- moved D27 5.00 mm to (6.00, 40.0)
- moved R71 5.00 mm to (18.0, 39.0)
- moved R46 2.24 mm to (24.0, 50.0)
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Routing:
- net DI3_LOGIC: track 118.5 -> 162.4 mm, vias 1 -> 2
- net ESP_BOOT: track 44.7 -> 85.8 mm
- net STATUS_GREEN_DRV: track 75.7 -> 35.1 mm, vias 5 -> 3
- net 3V3: track 428.1 -> 390.3 mm, vias 8 -> 6
- net STATUS_GREEN_K: track 44.7 -> 16.0 mm, vias 2 -> 3
- net SD_MISO: track 129.7 -> 104.4 mm, vias 5 -> 3
- net BUCK_FB: track 54.5 -> 37.1 mm, vias 3 -> 2
- net VIN_PROTECTED: track 112.9 -> 96.2 mm, vias 3 -> 5
- net STATUS_RED_K: track 31.3 -> 18.5 mm
- net 3V3A: track 90.3 -> 103.0 mm
- net SD_MOSI: track 107.2 -> 119.6 mm
- net STATUS_LED_CTL: track 48.8 -> 60.8 mm, vias 4 -> 3
- net ETH_LED_ACT_K: track 54.5 -> 65.0 mm
- net RTC_VDD: track 13.1 -> 23.1 mm, vias 0 -> 2
- net DI4_LOGIC: track 155.3 -> 165.2 mm
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